Commit message: Update pingu.urdf.xacro to adjust box size and material, and include arm descriptions

File: ros_ws/src/pingu_launch/description/urdf/pingu.urdf.xacro (robot description, xacro)
@@ -7,12 +7,16 @@
   <!-- Import RW ros2 control description -->
   <xacro:include filename="$(find rw_ros2_control)/ros2_control/rw.ros2_control.xacro" />
+  <!-- Import arm description -->
+    <!-- Include materials -->
+  <xacro:include filename="$(find levion_arm_ros2_control)/config/material.macros.xacro"/>
+  <xacro:include filename="$(find levion_arm_ros2_control)/urdf/levion_arm.macros.xacro"/>
   <!-- Base description -->
   <link name="base_link">
     <visual>
       <geometry>
-        <box size="0.1 0.1 0.1"/>
+        <box size="0.4 0.4 0.6"/>
       </geometry>
-      <material name="blue">
-        <color rgba="0 0 1 1"/>
+      <material name="black_transparent">
+        <color rgba="0 0 0 0.5"/>
       </material>
     </visual>
@@ -34,4 +38,11 @@
     <origin xyz="0 0 0" rpy="0 0 0" />
   </xacro:rw>
+  <!-- Arm description -->
+  <xacro:levion_arm parent="base_link" prefix="$(arg prefix)" left_right="left">
+    <origin xyz="0 0 0" rpy="0 0 0" />
+  </xacro:levion_arm>
+  <xacro:levion_arm parent="base_link" prefix="$(arg prefix)" left_right="right">
+    <origin xyz="0 0 0" rpy="0 0 0" />
+  </xacro:levion_arm>
   <!-- RW ros2 control description -->
   <xacro:rw_system name="RwSystem" prefix="$(arg prefix)"/>

Commit message: Add levion property configuration and update URDF for arm orientation and dimensions

File: ros_ws/src/pingu_launch/description/urdf/pingu.urdf.xacro (robot description, xacro)
@@ -9,4 +9,5 @@
   <!-- Import arm description -->
   <xacro:include filename="$(find levion_arm_ros2_control)/config/material.macros.xacro"/>
+  <xacro:include filename="$(find levion_arm_ros2_control)/config/levion.property.xacro"/>
   <xacro:include filename="$(find levion_arm_ros2_control)/urdf/levion_arm.macros.xacro"/>
   <xacro:include filename="$(find levion_arm_ros2_control)/ros2_control/levion_arm.ros2_control.xacro"/>
@@ -20,13 +21,15 @@
         <color rgba="0 0 0 0.5"/>
       </material>
+      <origin xyz="0 0 0" rpy="0 0 ${PI/2}"/>
     </visual>
     <collision>
       <geometry>
-        <box size="0.1 0.1 0.1"/>
+        <box size="0.4 0.4 0.6"/>
       </geometry>
+      <origin xyz="0 0 0" rpy="0 0 ${PI/2}"/>
     </collision>
     <inertial>
       <mass value="1.0"/>
-      <origin xyz="0 0 0" rpy="0 0 0"/>
+      <origin xyz="0 0 0" rpy="0 0 ${PI/2}"/>
       <inertia ixx="0.01" ixy="0" ixz="0" iyy="0.01" iyz="0" izz="0.01"/>
     </inertial>
@@ -40,8 +43,8 @@
   <!-- Arm description -->
   <xacro:levion_arm parent="base_link" prefix="$(arg prefix)" left_right="left">
-    <origin xyz="0 0 0" rpy="0 0 0" />
+    <origin xyz="0 0 0" rpy="0 0 ${-PI/2}" />
   </xacro:levion_arm>
   <xacro:levion_arm parent="base_link" prefix="$(arg prefix)" left_right="right">
-    <origin xyz="0 0 0" rpy="0 0 0" />
+    <origin xyz="0 0 0" rpy="0 0 ${PI/2}" />
   </xacro:levion_arm>
   <!-- RW ros2 control description -->

Commit message: Update robot orientation in URDF for base and arms to correct positioning

File: ros_ws/src/pingu_launch/description/urdf/pingu.urdf.xacro (robot description, xacro)
@@ -21,5 +21,5 @@
         <color rgba="0 0 0 0.5"/>
       </material>
-      <origin xyz="0 0 0" rpy="0 0 ${PI/2}"/>
+      <origin xyz="0 0 0" rpy="0 0 ${PI/4}"/>
     </visual>
     <collision>
@@ -27,9 +27,9 @@
         <box size="0.4 0.4 0.6"/>
       </geometry>
-      <origin xyz="0 0 0" rpy="0 0 ${PI/2}"/>
+      <origin xyz="0 0 0" rpy="0 0 ${PI/4}"/>
     </collision>
     <inertial>
       <mass value="1.0"/>
-      <origin xyz="0 0 0" rpy="0 0 ${PI/2}"/>
+      <origin xyz="0 0 0" rpy="0 0 ${PI/4}"/>
       <inertia ixx="0.01" ixy="0" ixz="0" iyy="0.01" iyz="0" izz="0.01"/>
     </inertial>
@@ -43,8 +43,8 @@
   <!-- Arm description -->
   <xacro:levion_arm parent="base_link" prefix="$(arg prefix)" left_right="left">
-    <origin xyz="0 0 0" rpy="0 0 ${-PI/2}" />
+    <origin xyz="${.28*SQRT2_2} ${.28*SQRT2_2} 0" rpy="0 0 ${PI/4}" />
   </xacro:levion_arm>
   <xacro:levion_arm parent="base_link" prefix="$(arg prefix)" left_right="right">
-    <origin xyz="0 0 0" rpy="0 0 ${PI/2}" />
+    <origin xyz="${.28*SQRT2_2} ${-.28*SQRT2_2} 0" rpy="0 0 ${-PI/4}" />
   </xacro:levion_arm>
   <!-- RW ros2 control description -->

Commit message: Refactor URDF generation and export process to support launch arguments for robot configuration

File: ros_ws/src/pingu_launch/description/urdf/pingu.urdf.xacro (robot description, xacro)
@@ -1,14 +1,21 @@
 <?xml version="1.0"?>
-<robot xmlns:xacro="http://www.ros.org/wiki/xacro" name="2dof_robot">
+<robot xmlns:xacro="http://www.ros.org/wiki/xacro" name="pingu">
   <!-- Enable setting arguments from the launch file -->
   <xacro:arg name="prefix" default="" />
+  <xacro:arg name="ros2_control" default="true" /> <!-- Enable ros2 control -->
+  <xacro:arg name="left_arm" default="true" />     <!-- Enable left arm -->
+  <xacro:arg name="right_arm" default="true" />    <!-- Enable right arm -->
   <!-- Import RW description -->
   <xacro:include filename="$(find rw_ros2_control)/urdf/rw.macro.xacro" />
   <!-- Import RW ros2 control description -->
-  <xacro:include filename="$(find rw_ros2_control)/ros2_control/rw.ros2_control.xacro" />
+  <xacro:if value="$(arg ros2_control)">
+    <xacro:include filename="$(find rw_ros2_control)/ros2_control/rw.ros2_control.xacro" />
+  </xacro:if>
+  <!-- TODO: Make it possible to skip if not needed -->
   <!-- Import arm description -->
   <xacro:include filename="$(find levion_arm_ros2_control)/config/material.macros.xacro"/>
   <xacro:include filename="$(find levion_arm_ros2_control)/config/levion.property.xacro"/>
   <xacro:include filename="$(find levion_arm_ros2_control)/urdf/levion_arm.macros.xacro"/>
+  <!-- Import arm ros2 control -->
   <xacro:include filename="$(find levion_arm_ros2_control)/ros2_control/levion_arm.ros2_control.xacro"/>
   <!-- Base description -->
@@ -42,13 +49,18 @@
   </xacro:rw>
   <!-- Arm description -->
-  <xacro:levion_arm parent="base_link" prefix="$(arg prefix)" left_right="left">
-    <origin xyz="${.28*SQRT2_2} ${.28*SQRT2_2} 0" rpy="0 0 ${PI/4}" />
-  </xacro:levion_arm>
-  <xacro:levion_arm parent="base_link" prefix="$(arg prefix)" left_right="right">
-    <origin xyz="${.28*SQRT2_2} ${-.28*SQRT2_2} 0" rpy="0 0 ${-PI/4}" />
-  </xacro:levion_arm>
-  <!-- RW ros2 control description -->
-  <xacro:rw_system name="RwSystem" prefix="$(arg prefix)"/>
-  <!-- Arm ros2 control description -->
-  <xacro:levion_system name="levion_arm" prefix="$(arg prefix)" left_arm="true" right_arm="true"/>
+  <xacro:if value="$(arg left_arm)">
+    <xacro:levion_arm parent="base_link" prefix="$(arg prefix)" left_right="left">
+      <origin xyz="${.28*SQRT2_2} ${.28*SQRT2_2} 0" rpy="0 0 ${PI/4}" />
+    </xacro:levion_arm>
+  </xacro:if>
+  <xacro:if value="$(arg right_arm)">
+    <xacro:levion_arm parent="base_link" prefix="$(arg prefix)" left_right="right">
+      <origin xyz="${.28*SQRT2_2} ${-.28*SQRT2_2} 0" rpy="0 0 ${-PI/4}" />
+    </xacro:levion_arm>
+  </xacro:if>
+  <!-- Ros2 control description -->
+  <xacro:if value="$(arg ros2_control)">
+    <xacro:rw_system name="RwSystem" prefix="$(arg prefix)"/>
+    <xacro:levion_system name="levion_arm" prefix="$(arg prefix)" left_arm="true" right_arm="true"/>
+  </xacro:if>
 </robot>

Commit message: Add base_link mesh and update URDF for visual and collision geometry

File: ros_ws/src/pingu_launch/description/urdf/pingu.urdf.xacro (robot description, xacro)
@@ -23,5 +23,5 @@
     <visual>
       <geometry>
-        <box size="0.4 0.4 0.6"/>
+        <mesh filename="package://pingu_launch/mesh/base_link.stl" scale="1 1 1"/>
       </geometry>
       <material name="black_transparent">
@@ -32,7 +32,7 @@
     <collision>
       <geometry>
-        <box size="0.4 0.4 0.6"/>
+        <box size="0.4 0.4 0.6552"/>
       </geometry>
-      <origin xyz="0 0 0" rpy="0 0 ${PI/4}"/>
+      <origin xyz="0 0 0.3276" rpy="0 0 ${PI/4}"/>
     </collision>
     <inertial>
@@ -46,15 +46,15 @@
   <!-- RW description -->
   <xacro:rw parent="base_link" prefix="$(arg prefix)">
-    <origin xyz="0 0 0" rpy="0 0 0" />
+    <origin xyz="0 0 .2875" rpy="0 0 0" />
   </xacro:rw>
   <!-- Arm description -->
   <xacro:if value="$(arg left_arm)">
     <xacro:levion_arm parent="base_link" prefix="$(arg prefix)" left_right="left">
-      <origin xyz="${.28*SQRT2_2} ${.28*SQRT2_2} 0" rpy="0 0 ${PI/4}" />
+      <origin xyz="${.28*SQRT2_2} ${.28*SQRT2_2} .2875" rpy="0 0 ${PI/4}" />
     </xacro:levion_arm>
   </xacro:if>
   <xacro:if value="$(arg right_arm)">
     <xacro:levion_arm parent="base_link" prefix="$(arg prefix)" left_right="right">
-      <origin xyz="${.28*SQRT2_2} ${-.28*SQRT2_2} 0" rpy="0 0 ${-PI/4}" />
+      <origin xyz="${.28*SQRT2_2} ${-.28*SQRT2_2} .2875" rpy="0 0 ${-PI/4}" />
     </xacro:levion_arm>
   </xacro:if>

Commit message: Update arm origin positions in URDF for left and right arms

File: ros_ws/src/pingu_launch/description/urdf/pingu.urdf.xacro (robot description, xacro)
@@ -51,10 +51,10 @@
   <xacro:if value="$(arg left_arm)">
     <xacro:levion_arm parent="base_link" prefix="$(arg prefix)" left_right="left">
-      <origin xyz="${.28*SQRT2_2} ${.28*SQRT2_2} .2875" rpy="0 0 ${PI/4}" />
+      <origin xyz="${.25*SQRT2_2} ${.25*SQRT2_2} .3475" rpy="0 0 ${PI/4}" />
     </xacro:levion_arm>
   </xacro:if>
   <xacro:if value="$(arg right_arm)">
     <xacro:levion_arm parent="base_link" prefix="$(arg prefix)" left_right="right">
-      <origin xyz="${.28*SQRT2_2} ${-.28*SQRT2_2} .2875" rpy="0 0 ${-PI/4}" />
+      <origin xyz="${.25*SQRT2_2} ${-.25*SQRT2_2} .3475" rpy="0 0 ${-PI/4}" />
     </xacro:levion_arm>
   </xacro:if>

Commit message: Update inertial properties and arm origin positions in URDF

File: ros_ws/src/pingu_launch/description/urdf/pingu.urdf.xacro (robot description, xacro)
@@ -37,7 +37,7 @@
     </collision>
     <inertial>
-      <mass value="1.0"/>
+      <mass value="23.0"/>
       <origin xyz="0 0 0" rpy="0 0 ${PI/4}"/>
-      <inertia ixx="0.01" ixy="0" ixz="0" iyy="0.01" iyz="0" izz="0.01"/>
+      <inertia ixx="0.5" ixy="0" ixz="0" iyy="0.5" iyz="0" izz="0.5"/>
     </inertial>
   </link>
@@ -51,10 +51,10 @@
   <xacro:if value="$(arg left_arm)">
     <xacro:levion_arm parent="base_link" prefix="$(arg prefix)" left_right="left">
-      <origin xyz="${.25*SQRT2_2} ${.25*SQRT2_2} .3475" rpy="0 0 ${PI/4}" />
+      <origin xyz="${.26*SQRT2_2} ${.26*SQRT2_2} .3475" rpy="0 0 ${PI/4}" />
     </xacro:levion_arm>
   </xacro:if>
   <xacro:if value="$(arg right_arm)">
     <xacro:levion_arm parent="base_link" prefix="$(arg prefix)" left_right="right">
-      <origin xyz="${.25*SQRT2_2} ${-.25*SQRT2_2} .3475" rpy="0 0 ${-PI/4}" />
+      <origin xyz="${.26*SQRT2_2} ${-.26*SQRT2_2} .3475" rpy="0 0 ${-PI/4}" />
     </xacro:levion_arm>
   </xacro:if>

Commit message: Update launch and URDF files to enable Mujoco hardware plugin support in ROS2 control

File: ros_ws/src/pingu_launch/description/urdf/pingu.urdf.xacro (robot description, xacro)
@@ -5,4 +5,5 @@
   <xacro:arg name="floating_joint" default="false" /> <!-- When experted to simulator -->
   <xacro:arg name="ros2_control" default="true" />    <!-- When controlling hardware -->
+  <xacro:arg name="hw_plugin" default="real" />       <!-- Choose hardware interface: real/mujoco -->
   <xacro:arg name="left_arm" default="true" />        <!-- Enable left arm -->
   <xacro:arg name="right_arm" default="true" />       <!-- Enable right arm -->
@@ -68,6 +69,6 @@
   <!-- Ros2 control description -->
   <xacro:if value="$(arg ros2_control)">
-    <xacro:rw_system name="RwSystem" prefix="$(arg prefix)"/>
-    <xacro:levion_system name="levion_arm" prefix="$(arg prefix)" left_arm="true" right_arm="true"/>
+    <xacro:rw_system name="RwSystem" prefix="$(arg prefix)" hw_plugin="$(arg hw_plugin)"/>
+    <xacro:levion_system name="levion_arm" prefix="$(arg prefix)" left_arm="true" right_arm="true" hw_plugin="$(arg hw_plugin)"/>
   </xacro:if>
 </robot>

File: ros_ws/src/rw_ros2_control/description/ros2_control/rw.ros2_control.xacro (robot description, xacro)
@@ -1,10 +1,18 @@
 <?xml version="1.0"?>
 <robot xmlns:xacro="http://www.ros.org/wiki/xacro">
-  <xacro:macro name="rw_system" params="name prefix">
+  <xacro:macro name="rw_system" params="name prefix hw_plugin:=real"> <!-- real/mujoco -->
     <ros2_control name="${name}" type="system">
-      <hardware>
-        <plugin>odrive_ros2_control_plugin/ODriveHardwareInterface</plugin>
-        <param name="can">can0</param>
-      </hardware>
+      <!-- Chose hardware interfaces -->
+      <xacro:if value="${hw_plugin == 'real'}">
+        <hardware>
+          <plugin>odrive_ros2_control_plugin/ODriveHardwareInterface</plugin>
+          <param name="can">can0</param>
+        </hardware>
+      </xacro:if>
+      <xacro:if value="${hw_plugin == 'mujoco'}">
+        <hardware>
+          <plugin>mujoco_ros2_control/MujocoSystem</plugin>
+        </hardware>
+      </xacro:if>
       <joint name="${prefix}rw_joint">
         <command_interface name="position">
