Commit message: Update box dimensions and joint origin in rw.macro.xacro for improved URDF representation

File: ros_ws/src/rw_ros2_control/description/urdf/rw.macro.xacro (robot description, xacro)
@@ -12,5 +12,5 @@
       <origin xyz="0 0 0" rpy="0 0 0"/>
       <geometry>
-        <box size="0.1 0.1 0.01"/>
+        <box size="0.2 0.2 0.05"/>
       </geometry>
     </collision>
@@ -18,5 +18,5 @@
       <origin xyz="0 0 0" rpy="0 0 0"/>
       <geometry>
-        <box size="0.1 0.1 0.01"/>
+        <box size="0.2 0.2 0.05"/>
       </geometry>
       <material name="orange"/>
@@ -58,5 +58,5 @@
     <parent link="${prefix}rw_base"/>
     <child link="${prefix}rw_rotor"/>
-    <origin xyz="0 0 0" rpy="0 0 0"/>
+    <origin xyz="0 0 0.05" rpy="0 0 0"/>
     <axis xyz="0 0 1"/>
     <limit effort="10.0" lower="-3.14" upper="3.14" velocity="1.0"/>

Commit message: Add mesh file for rw_base and update URDF to use mesh for collision and visual elements

File: ros_ws/src/rw_ros2_control/description/urdf/rw.macro.xacro (robot description, xacro)
@@ -12,16 +12,16 @@
       <origin xyz="0 0 0" rpy="0 0 0"/>
       <geometry>
-        <box size="0.2 0.2 0.05"/>
+        <mesh filename="package://rw_ros2_control/mesh/rw_base.stl" scale="1 1 1"/>
       </geometry>
     </collision>
     <visual>
-      <origin xyz="0 0 0" rpy="0 0 0"/>
+      <origin xyz="0 0 0" rpy="0 0 0.785"/>
       <geometry>
-        <box size="0.2 0.2 0.05"/>
+        <mesh filename="package://rw_ros2_control/mesh/rw_base.stl" scale="1 1 1"/>
       </geometry>
       <material name="orange"/>
     </visual>
     <inertial>
-      <origin xyz="0 0 0" rpy="0 0 0"/>
+      <origin xyz="0 0 0" rpy="0 0 0.785"/>
       <mass value="1.0"/>
       <inertia

Commit message: Update controller configuration to use 'joints' key and fix joint naming in URDF macro

File: ros_ws/src/rw_ros2_control/description/urdf/rw.macro.xacro (robot description, xacro)
@@ -2,5 +2,5 @@
 <robot xmlns:xacro="http://www.ros.org/wiki/xacro">
   <xacro:macro name="rw" params="parent prefix *origin">
-  <joint name="${prefix}base_joint" type="fixed">
+  <joint name="${prefix}rw_base_joint" type="fixed">
     <xacro:insert_block name="origin" />
     <parent link="${parent}"/>

Commit message: Feature/create models for sim (#46)
* Add launch file to export URDF from Xacro

* add px4-mpc to dockerrepositories

* Add acados installation intside the docker; used in px4-mpc

* temp

* temp

* temp

* temp

* temp

* Add export_ping launch file to generate and export URDF from Xacro

* Add docstring to export_ping.launch.py for clarity on URDF export process

* Refactor URDF generation and export process to support launch arguments for robot configuration

* Enable left and right arms in export_ping launch file

* Add initial README and URDF files for Pingu_Model

* Update README for Mujoco export instructions and add pingu.xml model definition

* Add section for URDF generation in README

* Add mesh file for rw_base and update URDF to use mesh for collision and visual elements

* Add base_link mesh and update URDF for visual and collision geometry

* Update arm origin positions in URDF for left and right arms

* Add base_link mesh file for URDF integration

* Update inertial properties and arm origin positions in URDF

* Add STL files for Link0, Link1, and Link2 in Mujoco assets

* Add export_mj_model function and URDF files with STL links for Pingu model

* Enhance export_mj_model function to modify MJCF output: add floor, lighting, and update mesh paths

* Update export_mj_model to handle both .STL and .stl file extensions; add base_link and rw_base STL files for URDF integration

* Refactor Pingu model URDF and XACRO files: add floating joint support, update mesh paths, and adjust inertial properties

* Enhance export_mj_model and pingu.xml: add autogenerated comments, set integrator options, and ensure correct mesh paths

* Refactor export_mj_model and pingu.xml: streamline autogenerated comments, add thruster sites, and ensure actuator definitions for enhanced model integration

* Enhance export_mj_model function: add comments for thruster placement and actuator integration, and improve code readability

* temp

* Refactor thruster placement in export_mj_model and pingu.xml: update thruster site positions to a circular arrangement and change site type to cylinder for improved visibility.

* Update thruster site positions in export_mj_model and pingu.xml: raise height to 0.3 for improved visibility and consistency.

* Refactor thruster sites in export_mj_model and pingu.xml: update site dimensions and types for improved visibility and consistency, and adjust actuator configurations.

* Update thruster actuator gear configurations in export_mj_model and pingu.xml for improved control precision.

* Add quaternion attributes to thruster sites in pingu.xml for improved orientation representation and update actuator definitions in export_mj_model.py.

* Update thruster configurations in export_mj_model.py and pingu.xml: flip adjacent thrusters and add gear specifications for improved control.

* Update gravity and contact parameters in export_mj_model.py and pingu.xml for improved simulation accuracy

* Add mocap body and sites to pingu.xml and export_mj_model.py for motion capture integration

* Update launch and URDF files to enable Mujoco hardware plugin support in ROS2 control

* Add Mujoco hardware plugin support and joint configurations in pingu.urdf for ROS2 control

* Add export script and MJCF model for Pingu with floor, lighting, and thruster configurations

* Add hw_plugin launch argument to support hardware plugin configuration

* Update controller configuration to use 'joints' key and fix joint naming in URDF macro

* Add new image to remember failsafe setting for px4

* Rename joint from base_joint to rw_base_joint for consistency in naming conventions

* Change package name from pingu_launch to pingu_ros2_control

* Add initial package structure and launch files for pingu_description

* Remove unused launch files and URDF descriptions from pingu_ros2_control package

* Remove temporary section and clean up README formatting

---------

Co-authored-by: ricard <ricardmarsalicastan@gmail.com>

File: ros_ws/src/rw_ros2_control/description/urdf/rw.macro.xacro (robot description, xacro)
@@ -2,5 +2,5 @@
 <robot xmlns:xacro="http://www.ros.org/wiki/xacro">
   <xacro:macro name="rw" params="parent prefix *origin">
-  <joint name="${prefix}base_joint" type="fixed">
+  <joint name="${prefix}rw_base_joint" type="fixed">
     <xacro:insert_block name="origin" />
     <parent link="${parent}"/>
@@ -12,16 +12,16 @@
       <origin xyz="0 0 0" rpy="0 0 0"/>
       <geometry>
-        <box size="0.2 0.2 0.05"/>
+        <mesh filename="package://rw_ros2_control/mesh/rw_base.stl" scale="1 1 1"/>
       </geometry>
     </collision>
     <visual>
-      <origin xyz="0 0 0" rpy="0 0 0"/>
+      <origin xyz="0 0 0" rpy="0 0 0.785"/>
       <geometry>
-        <box size="0.2 0.2 0.05"/>
+        <mesh filename="package://rw_ros2_control/mesh/rw_base.stl" scale="1 1 1"/>
       </geometry>
       <material name="orange"/>
     </visual>
     <inertial>
-      <origin xyz="0 0 0" rpy="0 0 0"/>
+      <origin xyz="0 0 0" rpy="0 0 0.785"/>
       <mass value="1.0"/>
       <inertia

File: ros_ws/src/rw_ros2_control/description/urdf/rw.urdf.xacro (robot description, xacro)
@@ -1,4 +1,4 @@
 <?xml version="1.0"?>
-<robot xmlns:xacro="http://www.ros.org/wiki/xacro" name="2dof_robot">
+<robot xmlns:xacro="http://www.ros.org/wiki/xacro" name="reaction_wheel">
   <!-- Enable setting arguments from the launch file -->
   <xacro:arg name="prefix" default="" />

Commit message: Update joint limits for rw_joint in rw.macro.xacro

File: ros_ws/src/rw_ros2_control/description/urdf/rw.macro.xacro (robot description, xacro)
@@ -60,5 +60,5 @@
     <origin xyz="0 0 0.05" rpy="0 0 0"/>
     <axis xyz="0 0 1"/>
-    <limit effort="10.0" lower="-3.14" upper="3.14" velocity="1.0"/>
+    <limit effort="10.0" lower="-1e9" upper="1e9" velocity="100"/>
     <dynamics damping="0.5" friction="0.5"/>
   </joint>
