Commit message: Update inertial properties of the base link in pingu.urdf.xacro

File: ros_ws/src/pingu_description/urdf/pingu.urdf.xacro (robot description, xacro)
@@ -48,6 +48,6 @@
     <inertial>
       <mass value="23.0"/>
-      <origin xyz="0 0 0" rpy="0 0 ${PI/4}"/>
-      <inertia ixx="0.5" ixy="0" ixz="0" iyy="0.5" iyz="0" izz="0.5"/>
+      <origin xyz="0 0 0.3276" rpy="0 0 ${PI/4}"/>
+      <inertia ixx="0.7" ixy="0" ixz="0" iyy="0.7" iyz="0" izz="0.5"/>
     </inertial>
   </link>

Commit message: Add launch arguments for left and right arm configuration in pingu.launch.py

File: ros_ws/src/pingu_description/urdf/pingu.urdf.xacro (robot description, xacro)
@@ -8,4 +8,12 @@
   <xacro:arg name="left_arm" default="true" />        <!-- Enable left arm -->
   <xacro:arg name="right_arm" default="true" />       <!-- Enable right arm -->
+  <!-- Check if it has arms-->
+  <xacro:property name="has_arm" value="false"/>
+  <xacro:if value="$(arg left_arm)">
+    <xacro:property name="has_arm" value="true"/>
+  </xacro:if>
+  <xacro:if value="$(arg right_arm)">
+    <xacro:property name="has_arm" value="true"/>
+  </xacro:if>
   <!-- Import RW description -->
   <xacro:include filename="$(find rw_ros2_control)/urdf/rw.macro.xacro" />
@@ -14,11 +22,13 @@
     <xacro:include filename="$(find rw_ros2_control)/ros2_control/rw.ros2_control.xacro" />
   </xacro:if>
-  <!-- TODO: Make it possible to skip if not needed -->
-  <!-- Import arm description -->
+  <!-- Import levion arm macros and properties -->
   <xacro:include filename="$(find levion_arm_ros2_control)/config/material.macros.xacro"/>
   <xacro:include filename="$(find levion_arm_ros2_control)/config/levion.property.xacro"/>
-  <xacro:include filename="$(find levion_arm_ros2_control)/urdf/levion_arm.macros.xacro"/>
-  <!-- Import arm ros2 control -->
-  <xacro:include filename="$(find levion_arm_ros2_control)/ros2_control/levion_arm.ros2_control.xacro"/>
+  <xacro:if value="${has_arm}">
+    <!-- Import arm description -->
+    <xacro:include filename="$(find levion_arm_ros2_control)/urdf/levion_arm.macros.xacro"/>
+    <!-- Import arm ros2 control -->
+    <xacro:include filename="$(find levion_arm_ros2_control)/ros2_control/levion_arm.ros2_control.xacro"/>
+  </xacro:if>
   <xacro:if value="$(arg floating_joint)">
     <link name="world"/>
@@ -70,5 +80,11 @@
   <xacro:if value="$(arg ros2_control)">
     <xacro:rw_system name="RwSystem" prefix="$(arg prefix)" hw_plugin="$(arg hw_plugin)"/>
-    <xacro:levion_system name="levion_arm" prefix="$(arg prefix)" left_arm="true" right_arm="true" hw_plugin="$(arg hw_plugin)"/>
+    <xacro:if value="${has_arm}">
+      <xacro:levion_system name="levion_arm"
+        prefix="$(arg prefix)"
+        left_arm="$(arg left_arm)"
+        right_arm="$(arg right_arm)"
+        hw_plugin="$(arg hw_plugin)"/>
+    </xacro:if>
   </xacro:if>
 </robot>

Commit message: Adjust RViz configuration and update URDF for fixed base joint; modify pose_to_tf to account for z-offset

File: ros_ws/src/pingu_description/urdf/pingu.urdf.xacro (robot description, xacro)
@@ -31,12 +31,20 @@
     <xacro:include filename="$(find levion_arm_ros2_control)/ros2_control/levion_arm.ros2_control.xacro"/>
   </xacro:if>
+  <!-- Define base_joint -->
+  <link name="world"/>
   <xacro:if value="$(arg floating_joint)">
-    <link name="world"/>
     <joint name="base_joint" type="floating">
-      <origin xyz="0 0 .2875" rpy="0 0 0"/>
+      <origin xyz="0 0 0" rpy="0 0 0"/>
       <parent link="world"/>
       <child link="base_link"/>
     </joint>
   </xacro:if>
+  <xacro:unless value="$(arg floating_joint)">
+    <joint name="base_joint" type="fixed">
+      <origin xyz="0 0 0.0" rpy="0 0 0"/>
+      <parent link="world"/>
+      <child link="base_link"/>
+    </joint>
+  </xacro:unless>
   <!-- Base description -->
   <link name="base_link">
