Commit message: pingu & cubo

File: ros_ws/src/pingu_description/urdf/pingu.urdf (robot description, URDF)
Before this commit: robot pingu_v3, 15 links, 14 joints
Links:
- added link left_link0, mass 0.5; collision mesh filename=package://pingu_description/mesh/arm_link0.stl scale=1 1 1; visual mesh filename=package://pingu_description/mesh/arm_link0.stl scale=1 1 1
- added link left_link1, mass 0.6; collision mesh filename=package://pingu_description/mesh/arm_link1.stl scale=1 1 1; visual mesh filename=package://pingu_description/mesh/arm_link1.stl scale=1 1 1
- added link left_link2, mass 0.1; collision mesh filename=package://pingu_description/mesh/arm_link2.stl scale=1 1 1; visual mesh filename=package://pingu_description/mesh/arm_link2.stl scale=1 1 1
- added link left_tool_link
- added link right_link0, mass 0.5; collision mesh filename=package://pingu_description/mesh/arm_link0.stl scale=1 1 1; visual mesh filename=package://pingu_description/mesh/arm_link0.stl scale=1 1 1
- added link right_link1, mass 0.6; collision mesh filename=package://pingu_description/mesh/arm_link1.stl scale=1 1 1; visual mesh filename=package://pingu_description/mesh/arm_link1.stl scale=1 1 1
- added link right_link2, mass 0.1; collision mesh filename=package://pingu_description/mesh/arm_link2.stl scale=1 1 1; visual mesh filename=package://pingu_description/mesh/arm_link2.stl scale=1 1 1
- added link right_tool_link
Joints:
- added joint left_base_joint: type fixed, parent base_link, child left_link0, origin xyz=0.26 0 .3475 rpy=0 0 0
- added joint left_elbow_joint: type revolute, parent left_link1, child left_link2, origin xyz=0.32 0 0.04685 rpy=0 0 0, axis 0 0 1, limit lower=-2.6050000000000004 upper=-0.359 effort=10 velocity=10
- added joint left_shoulder_joint: type revolute, parent left_link0, child left_link1, origin xyz=0 0 0.0439 rpy=0 0 0, axis 0 0 1, limit lower=-1.56079632675 upper=1.56079632675 effort=10 velocity=10
- added joint left_tool_joint: type fixed, parent left_link2, child left_tool_link, origin xyz=.255 0 0 rpy=1.57079632675 0 1.57079632675
- added joint right_base_joint: type fixed, parent base_link, child right_link0, origin xyz=0 -0.26 .3475 rpy=0 0 -1.57079632675
- added joint right_elbow_joint: type revolute, parent right_link1, child right_link2, origin xyz=0.32 0 0.04685 rpy=0 0 0, axis 0 0 1, limit lower=0.359 upper=2.6050000000000004 effort=10 velocity=10
- added joint right_shoulder_joint: type revolute, parent right_link0, child right_link1, origin xyz=0 0 0.0439 rpy=0 0 0, axis 0 0 1, limit lower=-1.56079632675 upper=1.56079632675 effort=10 velocity=10
- added joint right_tool_joint: type fixed, parent right_link2, child right_tool_link, origin xyz=.255 0 0 rpy=1.57079632675 0 1.57079632675

File: ros_ws/src/pingu_description/urdf/pingu_v3.urdf.xacro (robot description, xacro)
@@ -16,55 +16,19 @@
   <xacro:include filename="thruster/thruster.macro.xacro"/>
   <!-- Defaults -->
+   <xacro:property name="HEIGHT_FROM_GROUND" value="0.05"/>
   <xacro:property name="THRUSTER_OFFSET" value="0.168"/>
   <xacro:property name="THRUSTER_TOP" value="0.305"/>
   <xacro:property name="THRUSTER_BOTTOM" value="0.295"/>
+  <xacro:property name="Z_OFFSET" value="0.3"/>
   <!-- World Link -->
   <link name="world"/>
   <!-- Joins and Links for Floating -->
-  <link name="anchor_link">
-    <visual>
-      <geometry>
-        <box size="0.001 0.001 0.001"></box>
-      </geometry>
-      <material name="levion_black"/>
-      <origin xyz="0 0 0" rpy="0 0 0"/>
-    </visual>
-    <collision>
-      <geometry>
-        <box size="0.001 0.001 0.001"></box>
-      </geometry>
-      <origin xyz="0 0 0" rpy="0 0 0"/>
-    </collision>
-    <inertial>
-      <mass value="0.0001"/>
-      <origin xyz="0 0 0" rpy="0 0 0"/>
-      <inertia ixx="0.0001" ixy="0" ixz="0" iyy="0.0001" iyz="0" izz="0.0001"/>
-    </inertial>
-  </link>
+  <link name="anchor_link"/>
   <joint name="anchor_joint" type="fixed">
-    <origin xyz="0 0 0.2" rpy="0 0 0"/>
+    <origin xyz="0 0 ${HEIGHT_FROM_GROUND}" rpy="0 0 0"/>
     <parent link="world"/>
     <child link="anchor_link"/>
   </joint>
-  <link name="x_lock_link">
-    <visual>
-      <geometry>
-        <box size="0.001 0.001 0.001"></box>
-      </geometry>
-      <material name="levion_black"/>
-      <origin xyz="0 0 0" rpy="0 0 0"/>
-    </visual>
-    <collision>
-      <geometry>
-        <box size="0.001 0.001 0.001"></box>
-      </geometry>
-      <origin xyz="0 0 0" rpy="0 0 0"/>
-    </collision>
-    <inertial>
-      <mass value="0.0001"/>
-      <origin xyz="0 0 0" rpy="0 0 0"/>
-      <inertia ixx="0.0001" ixy="0" ixz="0" iyy="0.0001" iyz="0" izz="0.0001"/>
-    </inertial>
-  </link>
+  <link name="x_lock_link"/>
   <joint name="x_lock_joint" type="prismatic">
     <origin xyz="0 0 0" rpy="0 0 0"/>
@@ -74,24 +38,5 @@
     <limit effort="10.0" lower="-10" upper="10" velocity="10"/>
   </joint>
-  <link name="y_lock_link">
-    <visual>
-      <geometry>
-        <box size="0.001 0.001 0.001"></box>
-      </geometry>
-      <material name="levion_black"/>
-      <origin xyz="0 0 0" rpy="0 0 0"/>
-    </visual>
-    <collision>
-      <geometry>
-        <box size="0.001 0.001 0.001"></box>
-      </geometry>
-      <origin xyz="0 0 0" rpy="0 0 0"/>
-    </collision>
-    <inertial>
-      <mass value="0.0001"/>
-      <origin xyz="0 0 0" rpy="0 0 0"/>
-      <inertia ixx="0.0001" ixy="0" ixz="0" iyy="0.0001" iyz="0" izz="0.0001"/>
-    </inertial>
-  </link>
+  <link name="y_lock_link"/>
   <joint name="y_lock_joint" type="prismatic">
     <origin xyz="0 0 0" rpy="0 0 0"/>
@@ -102,6 +47,26 @@
   </joint>
   <!-- Base Join and Link-->
+  <link name="base_link">
+    <visual>
+      <geometry>
+        <mesh filename="package://pingu_description/mesh/base_link.stl" scale="0.001 0.001 0.001"/>
+      </geometry>
+      <material name="levion_black"/>
+      <origin xyz="0 0 0" rpy="0 0 ${-PI/2}"/>
+    </visual>
+    <collision>
+      <geometry>
+        <mesh filename="package://pingu_description/mesh/base_link.stl" scale="0.001 0.001 0.001"/>
+      </geometry>
+      <origin xyz="0 0 0" rpy="0 0  ${-PI/2}"/> <!-- 0 0 0.3276 for box -->
+    </collision>
+    <inertial>
+      <mass value="23.0"/>
+      <origin xyz="0 0 0.3276" rpy="0 0  ${-PI/2}"/>
+      <inertia ixx="0.7" ixy="0" ixz="0" iyy="0.7" iyz="0" izz="0.5"/>
+    </inertial>
+  </link>
   <joint name="base_joint" type="revolute">
-    <origin xyz="0 0 0.1" rpy="0 0 0"/>
+    <origin xyz="0 0 0" rpy="0 0 0"/>
     <parent link="y_lock_link"/>
     <child link="base_link"/>
@@ -110,24 +75,4 @@
     <!-- <dynamics damping="0.5" friction="0.0"/> -->
   </joint>
-  <link name="base_link">
-    <visual>
-      <geometry>
-        <mesh filename="package://pingu_description/mesh/base_link.stl" scale="0.001 0.001 0.001"/>
-      </geometry>
-      <material name="levion_black"/>
-      <origin xyz="0 0 0" rpy="0 0 0"/>
-    </visual>
-    <collision>
-      <geometry>
-        <mesh filename="package://pingu_description/mesh/base_link.stl" scale="0.001 0.001 0.001"/>
-      </geometry>
-      <origin xyz="0 0 0" rpy="0 0 0"/> <!-- 0 0 0.3276 for box -->
-    </collision>
-    <inertial>
-      <mass value="23.0"/>
-      <origin xyz="0 0 0.3276" rpy="0 0 0"/>
-      <inertia ixx="0.7" ixy="0" ixz="0" iyy="0.7" iyz="0" izz="0.5"/>
-    </inertial>
-  </link>
   <!-- RW description -->
   <xacro:rw parent="base_link" prefix="$(arg prefix)">
@@ -135,11 +80,11 @@
   </xacro:rw>
   <!-- Left Arm description -->
-  <!-- <xacro:levion_arm parent="base_link" prefix="$(arg prefix)" left_right="left">
+  <xacro:levion_arm parent="base_link" prefix="$(arg prefix)" left_right="left">
     <origin xyz="0.26 0 .3475" rpy="0 0 0" />
-  </xacro:levion_arm> -->
+  </xacro:levion_arm>
   <!-- Right Arm description -->
-  <!-- <xacro:levion_arm parent="base_link" prefix="$(arg prefix)" left_right="right">
+  <xacro:levion_arm parent="base_link" prefix="$(arg prefix)" left_right="right">
     <origin xyz="0 -0.26 .3475" rpy="0 0 ${-PI/2}" />
-  </xacro:levion_arm> -->
+  </xacro:levion_arm>
   <!-- Thrusters description -->
   <xacro:thruster prefix="thruster_1"
@@ -148,8 +93,8 @@
   <xacro:thruster prefix="thruster_2"
                   parent="base_link"
-                  xyz="-${THRUSTER_OFFSET} ${THRUSTER_OFFSET} ${THRUSTER_TOP}" rpy="${PI/2} 0 ${-PI/4}"/>
+                  xyz="-${THRUSTER_OFFSET} ${THRUSTER_OFFSET} ${THRUSTER_TOP}" rpy="${-PI/2} 0 ${PI/4}"/>
   <xacro:thruster prefix="thruster_3"
                   parent="base_link"
-                  xyz="${THRUSTER_OFFSET} ${THRUSTER_OFFSET} ${THRUSTER_BOTTOM}" rpy="${PI/2} 0 ${PI/4}"/>
+                  xyz="${THRUSTER_OFFSET} ${THRUSTER_OFFSET} ${THRUSTER_BOTTOM}" rpy="${-PI/2} 0 ${-PI/4}"/>
   <xacro:thruster prefix="thruster_4"
                   parent="base_link"
@@ -157,5 +102,5 @@
   <xacro:thruster prefix="thruster_5"
                   parent="base_link"
-                  xyz="${THRUSTER_OFFSET} -${THRUSTER_OFFSET} ${THRUSTER_TOP}" rpy="${PI/2} 0 ${-PI/4}"/>
+                  xyz="${THRUSTER_OFFSET} -${THRUSTER_OFFSET} ${THRUSTER_TOP}" rpy="${-PI/2} 0 ${PI/4}"/>
   <xacro:thruster prefix="thruster_6"
                   parent="base_link"
@@ -166,4 +111,4 @@
   <xacro:thruster prefix="thruster_8"
                   parent="base_link"
-                  xyz="-${THRUSTER_OFFSET} -${THRUSTER_OFFSET} ${THRUSTER_BOTTOM}" rpy="${PI/2} 0 ${PI/4}"/>
+                  xyz="-${THRUSTER_OFFSET} -${THRUSTER_OFFSET} ${THRUSTER_BOTTOM}" rpy="${-PI/2} 0 ${-PI/4}"/>
 </robot>

File: ros_ws/src/pingu_description/urdf/thruster/thruster.macro.xacro (robot description, xacro)
@@ -2,5 +2,5 @@
 <robot xmlns:xacro="http://www.ros.org/wiki/xacro">
   <xacro:macro name="thruster" params="parent prefix xyz rpy">
-  <!-- Base Link -->
+  <!-- Thruster Link -->
   <link  name="${prefix}_link">
     <visual>
