Commit message: Update export_mj_model to handle both .STL and .stl file extensions; add base_link and rw_base STL files for URDF integration

File: Pingu_Model/description/urdf/pingu.urdf (robot description, URDF)
Before this commit: robot pingu, 11 links, 10 joints
Links:
- link base_link: geometry collision box size=0.4 0.4 0.6552; visual mesh filename=/home/spacer/ros_ws/install/pingu_launch/share/pingu_launch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 scale=1 1 1
- link rw_base: geometry collision mesh filename=/home/spacer/ros_ws/install/rw_ros2_control/share/rw_ros2_c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 scale=1 1 1; visual mesh filename=/home/spacer/ros_ws/install/rw_ros2_control/share/rw_ros2_c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 scale=1 1 1
Joints:
- joint base_joint: origin xyz=0 0 0 rpy=0 0 0 -> xyz=0 0 .2875 rpy=0 0 0
- joint left_base_joint: origin xyz=0.19798989872200004 0.19798989872200004 0 rpy=0 0 0.785398163375 -> xyz=0.1767766952875 0.1767766952875 .3475 rpy=0 0 0.785398163375
- joint right_base_joint: origin xyz=0.19798989872200004 -0.19798989872200004 0 rpy=0 0 -0.785398163375 -> xyz=0.1767766952875 -0.1767766952875 .3475 rpy=0 0 -0.785398163375

Commit message: Refactor Pingu model URDF and XACRO files: add floating joint support, update mesh paths, and adjust inertial properties

File: Pingu_Model/description/urdf/pingu.urdf (robot description, URDF)
Before this commit: robot pingu, 11 links, 10 joints
Links:
- added link world
- link base_link: mass 1.0 -> 23.0; geometry collision mesh filename=package://pingu_launch/mesh/base_link.stl scale=1 1 1; visual mesh filename=package://pingu_launch/mesh/base_link.stl scale=1 1 1
- link left_link0: mass 0.1 -> 0.5; geometry collision mesh filename=package://levion_arm_ros2_control/mesh/Link0.STL scale=1 1 1; visual mesh filename=package://levion_arm_ros2_control/mesh/Link0.STL scale=1 1 1
- link left_link1: mass 0.1 -> 0.6; geometry collision mesh filename=package://levion_arm_ros2_control/mesh/Link1.STL scale=1 1 1; visual mesh filename=package://levion_arm_ros2_control/mesh/Link1.STL scale=1 1 1
- link left_link2: geometry collision mesh filename=package://levion_arm_ros2_control/mesh/Link2.STL scale=1 1 1; visual mesh filename=package://levion_arm_ros2_control/mesh/Link2.STL scale=1 1 1
- link right_link0: mass 0.1 -> 0.5; geometry collision mesh filename=package://levion_arm_ros2_control/mesh/Link0.STL scale=1 1 1; visual mesh filename=package://levion_arm_ros2_control/mesh/Link0.STL scale=1 1 1
- link right_link1: mass 0.1 -> 0.6; geometry collision mesh filename=package://levion_arm_ros2_control/mesh/Link1.STL scale=1 1 1; visual mesh filename=package://levion_arm_ros2_control/mesh/Link1.STL scale=1 1 1
- link right_link2: geometry collision mesh filename=package://levion_arm_ros2_control/mesh/Link2.STL scale=1 1 1; visual mesh filename=package://levion_arm_ros2_control/mesh/Link2.STL scale=1 1 1
- link rw_base: geometry collision mesh filename=package://rw_ros2_control/mesh/rw_base.stl scale=1 1 1; visual mesh filename=package://rw_ros2_control/mesh/rw_base.stl scale=1 1 1
Joints:
- joint left_base_joint: origin xyz=0.1767766952875 0.1767766952875 .3475 rpy=0 0 0.785398163375 -> xyz=0.18384776309900003 0.18384776309900003 .3475 rpy=0 0 0.785398163375
- joint right_base_joint: origin xyz=0.1767766952875 -0.1767766952875 .3475 rpy=0 0 -0.785398163375 -> xyz=0.18384776309900003 -0.18384776309900003 .3475 rpy=0 0 -0.785398163375

File: ros_ws/src/pingu_launch/description/urdf/pingu.urdf.xacro (robot description, xacro)
@@ -3,7 +3,8 @@
   <!-- Enable setting arguments from the launch file -->
   <xacro:arg name="prefix" default="" />
-  <xacro:arg name="ros2_control" default="true" /> <!-- Enable ros2 control -->
-  <xacro:arg name="left_arm" default="true" />     <!-- Enable left arm -->
-  <xacro:arg name="right_arm" default="true" />    <!-- Enable right arm -->
+  <xacro:arg name="floating_joint" default="false" /> <!-- When experted to simulator -->
+  <xacro:arg name="ros2_control" default="true" />    <!-- When controlling hardware -->
+  <xacro:arg name="left_arm" default="true" />        <!-- Enable left arm -->
+  <xacro:arg name="right_arm" default="true" />       <!-- Enable right arm -->
   <!-- Import RW description -->
   <xacro:include filename="$(find rw_ros2_control)/urdf/rw.macro.xacro" />
@@ -19,4 +20,12 @@
   <!-- Import arm ros2 control -->
   <xacro:include filename="$(find levion_arm_ros2_control)/ros2_control/levion_arm.ros2_control.xacro"/>
+  <xacro:if value="$(arg floating_joint)">
+    <link name="world"/>
+    <joint name="base_joint" type="floating">
+      <origin xyz="0 0 .2875" rpy="0 0 0"/>
+      <parent link="world"/>
+      <child link="base_link"/>
+    </joint>
+  </xacro:if>
   <!-- Base description -->
   <link name="base_link">
@@ -32,7 +41,7 @@
     <collision>
       <geometry>
-        <box size="0.4 0.4 0.6552"/>
+        <mesh filename="package://pingu_launch/mesh/base_link.stl" scale="1 1 1"/>
       </geometry>
-      <origin xyz="0 0 0.3276" rpy="0 0 ${PI/4}"/>
+      <origin xyz="0 0 0" rpy="0 0 ${PI/4}"/> <!-- 0 0 0.3276 for box -->
     </collision>
     <inertial>
@@ -42,6 +51,4 @@
     </inertial>
   </link>
-  <!-- Used for fixing robot -->
-  <!-- <link name="world"/> -->
   <!-- RW description -->
   <xacro:rw parent="base_link" prefix="$(arg prefix)">

Commit message: Change package name from pingu_launch to pingu_ros2_control

File: Pingu_Model/description/urdf/pingu.urdf (robot description, URDF)
Before this commit: robot pingu, 12 links, 11 joints
Links:
- link base_link: geometry collision mesh filename=package://pingu_ros2_control/mesh/base_link.stl scale=1 1 1; visual mesh filename=package://pingu_ros2_control/mesh/base_link.stl scale=1 1 1

File: ros_ws/src/pingu_ros2_control/description/urdf/pingu.urdf.xacro (robot description, xacro)
@@ -33,5 +33,5 @@
     <visual>
       <geometry>
-        <mesh filename="package://pingu_launch/mesh/base_link.stl" scale="1 1 1"/>
+        <mesh filename="package://pingu_ros2_control/mesh/base_link.stl" scale="1 1 1"/>
       </geometry>
       <material name="black_transparent">
@@ -42,5 +42,5 @@
     <collision>
       <geometry>
-        <mesh filename="package://pingu_launch/mesh/base_link.stl" scale="1 1 1"/>
+        <mesh filename="package://pingu_ros2_control/mesh/base_link.stl" scale="1 1 1"/>
       </geometry>
       <origin xyz="0 0 0" rpy="0 0 ${PI/4}"/> <!-- 0 0 0.3276 for box -->

Commit message: Update inertial properties and joint limits in pingu model

File: Pingu_Model/description/urdf/pingu.urdf (robot description, URDF)
Before this commit: robot pingu, 12 links, 11 joints
Links:
- link base_link: geometry collision mesh filename=package://pingu_description/mesh/base_link.stl scale=1 1 1; visual mesh filename=package://pingu_description/mesh/base_link.stl scale=1 1 1
Joints:
- joint rw_joint: limit lower=-3.14 upper=3.14 effort=10.0 velocity=1.0 -> lower=-1e9 upper=1e9 effort=10.0 velocity=100

Commit message: Update inertial properties in pingu model and rw_joint definitions

File: Pingu_Model/description/urdf/pingu.urdf (robot description, URDF)
Before this commit: robot pingu, 12 links, 11 joints
Links:
- link rw_rotor: mass 1.0 -> 2.0

File: ros_ws/src/rw_ros2_control/description/urdf/rw.macro.xacro (robot description, xacro)
@@ -26,7 +26,7 @@
       <mass value="1.0"/>
       <inertia
-        ixx="0.06" ixy="0.0" ixz="0.0"
-        iyy="0.06" iyz="0.0"
-        izz="0.1"/>
+        ixx="0.01" ixy="0.0" ixz="0.0"
+        iyy="0.01" iyz="0.0"
+        izz="0.01"/>
     </inertial>
   </link>
@@ -48,9 +48,9 @@
     <inertial>
       <origin xyz="0 0 0" rpy="0 0 0"/>
-      <mass value="1.0"/>
+      <mass value="2.0"/>
       <inertia
-        ixx="0.0001" ixy="0.0" ixz="0.0"
-        iyy="0.0001" iyz="0.0"
-        izz="0.0001"/>
+        ixx="0.06" ixy="0.0" ixz="0.0"
+        iyy="0.06" iyz="0.0"
+        izz="0.1"/>
     </inertial>
   </link>

Commit message: Akiyoshi/setup thruster eval (#47)
* Add documentation for ZeroG Lab and Jetson setup

* Add command interfaces for velocity and effort in rw.ros2_control.xacro

* Update joint limits for rw_joint in rw.macro.xacro

* Update inertial properties of the base link in pingu.urdf.xacro

* Update inertial properties and joint limits in pingu model

* Update inertial properties and mesh content types in pingu model

* Remove content_type attributes from mesh definitions in pingu.xml

* Update inertial properties in pingu model and rw_joint definitions

* Update base_link STL files in pingu model

* Add keyboard valve control node and update setup entry points

* Add actuator controllers to configuration and update launch file

* Fix controller type casing in actuator configuration

* Update TODO comment to clarify controller selection for spawning

* Update spawner arguments to use position controller instead of velocity controller

* Refactor URDF export logic by encapsulating XACRO parsing and URI resolution in a dedicated function

* Add actuators trajectory controller configuration with parameters and gains

* Comment out actuators trajectory controller spawner node in launch file

* Add initial bashrc configuration with custom settings and aliases

* Add rosbag

* Initialize pingu_optitrack package with essential files and configurations

* Enhance documentation and launch configuration for actuator control

- Updated zeroG.md to include detailed options for launching actuators.
- Modified pingu.launch.py to support dynamic controller spawners.
- Added Gazebo hardware plugin option in rw.ros2_control.xacro.

* Add launch arguments for left and right arm configuration in pingu.launch.py

* Add controller spawners to launch description

* Update zeroG.md to include specific controller options for launching actuators

* Adjust RViz configuration and update URDF for fixed base joint; modify pose_to_tf to account for z-offset

* Update RViz configuration: add grid panel, adjust grid color and offset, modify view parameters

* Add zero_g robot description and update RViz configuration for visualization

* Update RViz configuration: remove unused panels, disable all frames, and adjust focal point and view parameters

* Fix thruster positions and update mocap body position in MJCF model

* Add new rosbag file for data collection on 2025-06-20

* Add new rosbag file for data collection on 2025-06-20

* Add new rosbag file for data collection on 2025-06-20

* Add new rosbag file for data collection on 2025-06-20

* Add new rosbag file for data collection on 2025-06-20

* Add new rosbag file for data collection on 2025-06-20 at 17:29:41

* Add new rosbag file for data collection on 2025-06-20 at 17:32:24

* Add new rosbag file for data collection on 2025-06-20 at 17:34:23

* Add new rosbag file for MPC test data collection

* Remove outdated rosbag files from June 19 and June 20, 2025

* Fix formatting and update launch command for Rviz in zeroG documentation

* Refactor keyboard input handling in KeyboardPublisher to use terminal settings instead of threading

* Fix timestamp assignment in TransformStamped to use message header

* Add model documentation and update launch configuration for ZeroG support

---------

Co-authored-by: ricard <ricardmarsalicastan@gmail.com>

File: Pingu_Model/description/urdf/pingu.urdf (robot description, URDF)
Before this commit: robot pingu, 12 links, 11 joints
Links:
- link base_link: geometry collision mesh filename=package://pingu_description/mesh/base_link.stl scale=1 1 1; visual mesh filename=package://pingu_description/mesh/base_link.stl scale=1 1 1
- link rw_rotor: mass 1.0 -> 2.0
Joints:
- joint rw_joint: limit lower=-3.14 upper=3.14 effort=10.0 velocity=1.0 -> lower=-1e9 upper=1e9 effort=10.0 velocity=100

File: ros_ws/src/pingu_description/urdf/pingu.urdf.xacro (robot description, xacro)
@@ -8,4 +8,12 @@
   <xacro:arg name="left_arm" default="true" />        <!-- Enable left arm -->
   <xacro:arg name="right_arm" default="true" />       <!-- Enable right arm -->
+  <!-- Check if it has arms-->
+  <xacro:property name="has_arm" value="false"/>
+  <xacro:if value="$(arg left_arm)">
+    <xacro:property name="has_arm" value="true"/>
+  </xacro:if>
+  <xacro:if value="$(arg right_arm)">
+    <xacro:property name="has_arm" value="true"/>
+  </xacro:if>
   <!-- Import RW description -->
   <xacro:include filename="$(find rw_ros2_control)/urdf/rw.macro.xacro" />
@@ -14,19 +22,29 @@
     <xacro:include filename="$(find rw_ros2_control)/ros2_control/rw.ros2_control.xacro" />
   </xacro:if>
-  <!-- TODO: Make it possible to skip if not needed -->
-  <!-- Import arm description -->
+  <!-- Import levion arm macros and properties -->
   <xacro:include filename="$(find levion_arm_ros2_control)/config/material.macros.xacro"/>
   <xacro:include filename="$(find levion_arm_ros2_control)/config/levion.property.xacro"/>
-  <xacro:include filename="$(find levion_arm_ros2_control)/urdf/levion_arm.macros.xacro"/>
-  <!-- Import arm ros2 control -->
-  <xacro:include filename="$(find levion_arm_ros2_control)/ros2_control/levion_arm.ros2_control.xacro"/>
+  <xacro:if value="${has_arm}">
+    <!-- Import arm description -->
+    <xacro:include filename="$(find levion_arm_ros2_control)/urdf/levion_arm.macros.xacro"/>
+    <!-- Import arm ros2 control -->
+    <xacro:include filename="$(find levion_arm_ros2_control)/ros2_control/levion_arm.ros2_control.xacro"/>
+  </xacro:if>
+  <!-- Define base_joint -->
+  <link name="world"/>
   <xacro:if value="$(arg floating_joint)">
-    <link name="world"/>
     <joint name="base_joint" type="floating">
-      <origin xyz="0 0 .2875" rpy="0 0 0"/>
+      <origin xyz="0 0 0" rpy="0 0 0"/>
       <parent link="world"/>
       <child link="base_link"/>
     </joint>
   </xacro:if>
+  <xacro:unless value="$(arg floating_joint)">
+    <joint name="base_joint" type="fixed">
+      <origin xyz="0 0 0.0" rpy="0 0 0"/>
+      <parent link="world"/>
+      <child link="base_link"/>
+    </joint>
+  </xacro:unless>
   <!-- Base description -->
   <link name="base_link">
@@ -48,6 +66,6 @@
     <inertial>
       <mass value="23.0"/>
-      <origin xyz="0 0 0" rpy="0 0 ${PI/4}"/>
-      <inertia ixx="0.5" ixy="0" ixz="0" iyy="0.5" iyz="0" izz="0.5"/>
+      <origin xyz="0 0 0.3276" rpy="0 0 ${PI/4}"/>
+      <inertia ixx="0.7" ixy="0" ixz="0" iyy="0.7" iyz="0" izz="0.5"/>
     </inertial>
   </link>
@@ -70,5 +88,11 @@
   <xacro:if value="$(arg ros2_control)">
     <xacro:rw_system name="RwSystem" prefix="$(arg prefix)" hw_plugin="$(arg hw_plugin)"/>
-    <xacro:levion_system name="levion_arm" prefix="$(arg prefix)" left_arm="true" right_arm="true" hw_plugin="$(arg hw_plugin)"/>
+    <xacro:if value="${has_arm}">
+      <xacro:levion_system name="levion_arm"
+        prefix="$(arg prefix)"
+        left_arm="$(arg left_arm)"
+        right_arm="$(arg right_arm)"
+        hw_plugin="$(arg hw_plugin)"/>
+    </xacro:if>
   </xacro:if>
 </robot>

File: ros_ws/src/rw_ros2_control/description/ros2_control/rw.ros2_control.xacro (robot description, xacro)
@@ -15,8 +15,21 @@
         </hardware>
       </xacro:if>
+      <xacro:if value="${hw_plugin == 'gazebo'}">
+        <hardware>
+          <plugin>gazebo_ros2_control/GazeboSystem</plugin>
+        </hardware>
+      </xacro:if>
       <joint name="${prefix}rw_joint">
         <command_interface name="position">
           <param name="min">-1</param>
           <param name="max">1</param>
+        </command_interface>
+        <command_interface name="velocity">
+          <param name="min">-10</param>
+          <param name="max">10</param>
+        </command_interface>
+        <command_interface name="effort">
+          <param name="min">-10</param>
+          <param name="max">10</param>
         </command_interface>
         <state_interface name="position"/>

File: ros_ws/src/rw_ros2_control/description/urdf/rw.macro.xacro (robot description, xacro)
@@ -26,7 +26,7 @@
       <mass value="1.0"/>
       <inertia
-        ixx="0.0001" ixy="0.0" ixz="0.0"
-        iyy="0.0001" iyz="0.0"
-        izz="0.0001"/>
+        ixx="0.01" ixy="0.0" ixz="0.0"
+        iyy="0.01" iyz="0.0"
+        izz="0.01"/>
     </inertial>
   </link>
@@ -48,9 +48,9 @@
     <inertial>
       <origin xyz="0 0 0" rpy="0 0 0"/>
-      <mass value="1.0"/>
+      <mass value="2.0"/>
       <inertia
-        ixx="0.0001" ixy="0.0" ixz="0.0"
-        iyy="0.0001" iyz="0.0"
-        izz="0.0001"/>
+        ixx="0.06" ixy="0.0" ixz="0.0"
+        iyy="0.06" iyz="0.0"
+        izz="0.1"/>
     </inertial>
   </link>
@@ -60,5 +60,5 @@
     <origin xyz="0 0 0.05" rpy="0 0 0"/>
     <axis xyz="0 0 1"/>
-    <limit effort="10.0" lower="-3.14" upper="3.14" velocity="1.0"/>
+    <limit effort="10.0" lower="-1e9" upper="1e9" velocity="100"/>
     <dynamics damping="0.5" friction="0.5"/>
   </joint>
