Commit message: UniLu FP with minimalist meshes

File: ros_ws/src/pingu_description/urdf/arms/levion_arm.macros.xacro (robot description, xacro)
@@ -13,4 +13,5 @@
     <xacro:property name="lr_elbow_vel" default="${left_elbow_velocity_limit}" />
     <xacro:property name="lr_elbow_effort" default="${left_elbow_effort_limit}" />
+    <xacro:property name="lr_link2_roll" default="${PI}" />
   </xacro:if>
   <xacro:if value="${left_right == 'right'}">
@@ -23,4 +24,5 @@
     <xacro:property name="lr_elbow_vel" default="${right_elbow_velocity_limit}" />
     <xacro:property name="lr_elbow_effort" default="${right_elbow_effort_limit}" />
+    <xacro:property name="lr_link2_roll" default="0" />
   </xacro:if>
   <joint name="${prefix}${left_right}_base_joint" type="fixed">
@@ -33,5 +35,5 @@
       <origin xyz="0 0 0" rpy="0 0 0"/>
       <geometry>
-        <mesh filename="package://pingu_description/mesh/arm_link0.stl" scale="1 1 1"/>
+        <mesh filename="package://pingu_description/mesh/arm_link_0.stl" scale="1 1 1"/>
       </geometry>
       <material name="levion_black"/>
@@ -40,5 +42,5 @@
       <origin xyz="0 0 0" rpy="0 0 0"/>
       <geometry>
-        <mesh filename="package://pingu_description/mesh/arm_link0.stl" scale="1 1 1"/>
+        <mesh filename="package://pingu_description/mesh/arm_link_0.stl" scale="1 1 1"/>
       </geometry>
     </collision>
@@ -53,5 +55,5 @@
       <origin xyz="0 0 0" rpy="0 0 0"/>
       <geometry>
-        <mesh filename="package://pingu_description/mesh/arm_link1.stl" scale="1 1 1"/>
+        <mesh filename="package://pingu_description/mesh/arm_link_1.stl" scale="1 1 1"/>
       </geometry>
       <material name="levion_black"/>
@@ -60,5 +62,5 @@
       <origin xyz="0 0 0" rpy="0 0 0"/>
       <geometry>
-        <mesh filename="package://pingu_description/mesh/arm_link1.stl" scale="1 1 1"/>
+        <mesh filename="package://pingu_description/mesh/arm_link_1.stl" scale="1 1 1"/>
       </geometry>
     </collision>
@@ -71,14 +73,14 @@
   <link name="${prefix}${left_right}_link2">
     <visual>
-      <origin xyz="0 0 0" rpy="0 0 0"/>
+      <origin xyz="0 0 0" rpy="${lr_link2_roll} 0 0"/>
       <geometry>
-        <mesh filename="package://pingu_description/mesh/arm_link2.stl" scale="1 1 1"/>
+        <mesh filename="package://pingu_description/mesh/arm_link_2.stl" scale="1 1 1"/>
       </geometry>
       <material name="levion_black"/>
     </visual>
     <collision>
-      <origin xyz="0 0 0" rpy="0 0 0"/>
+      <origin xyz="0 0 0" rpy="${lr_link2_roll} 0 0"/>
       <geometry>
-        <mesh filename="package://pingu_description/mesh/arm_link2.stl" scale="1 1 1"/>
+        <mesh filename="package://pingu_description/mesh/arm_link_2.stl" scale="1 1 1"/>
       </geometry>
     </collision>

File: ros_ws/src/pingu_description/urdf/rw/rw.macro.xacro (robot description, xacro)
@@ -3,5 +3,13 @@
   <xacro:macro name="rw" params="parent prefix *origin">
   <!-- Base Link -->
-  <link name="${prefix}rw_base" />
+  <link name="${prefix}rw_base">
+    <visual>
+      <origin xyz="0 0 0" rpy="0 0 0"/>
+      <geometry>
+        <mesh filename="package://pingu_description/mesh/minimalist_motor_holder.stl" scale="0.001 0.001 0.001"/>
+      </geometry>
+      <material name="levion_black"/>
+    </visual>
+  </link>
   <joint name="${prefix}rw_base_joint" type="fixed">
     <xacro:insert_block name="origin" />
@@ -14,5 +22,5 @@
       <origin xyz="0 0 0" rpy="0 0 0"/>
       <geometry>
-        <cylinder radius="0.1" length="0.008"/>
+        <mesh filename="package://pingu_description/mesh/minimalist_reaction_wheel.stl" scale="0.001 0.001 0.001"/>
       </geometry>
       <material name="orange"/>
@@ -20,5 +28,5 @@
     <inertial>
       <origin xyz="0 0 0" rpy="0 0 0"/>
-      <mass value="2.0"/>
+      <mass value="0.172"/>
       <inertia
         ixx="0.06" ixy="0.0" ixz="0.0"
