Commit message: Add setup scripts for ROS workspace and update Docker run configuration
- Created `setup.sh` and `setup.zsh` scripts to extend the environment for ROS packages.
- Added `COLCON_IGNORE` file in the log directory to ignore specific packages during build.
- Created symbolic links for `latest` and `latest_build` in the log directory to track the most recent build.
- Updated `run.sh` to improve X11 forwarding setup for Docker containers, ensuring proper DISPLAY and XAUTHORITY handling.
- Modified volume mounts in Docker run command to reflect new directory structure.
- Updated submodule reference for `LevionArm` to the latest commit.
- Changed `reaction_wheel` configuration in `pingu_config.yaml` to false.
- Enhanced `pingu_controllers.yaml` with additional arm controllers and improved comments.
- Refactored `pingu_low_level_controller_individual_thruster_control_launch.py` to support new arm controller arguments.
- Updated `pingu_low_level_controller_node.py` to handle new arm controllers and improve command handling.
- Adjusted URDF properties for arms to reflect new joint limits and configurations.
- Enhanced `pingu.urdf.xacro` to include new arguments for shoulder and elbow motors.
- Updated `rw.ros2_control.xacro` to accommodate new hardware interface options.

File: ros_ws/src/pingu_description/urdf/arms/levion.property.xacro (robot description, xacro)
@@ -12,6 +12,6 @@
   <!-- Default -->
   <xacro:property name="default_joint_position_limit" value="${PI/2-SAFETY_OFFSET}"/>
-  <xacro:property name="default_joint_velocity_limit" value="10"/>
-  <xacro:property name="default_joint_effort_limit" value="10"/>
+  <xacro:property name="default_joint_velocity_limit" value="1.0"/>
+  <xacro:property name="default_joint_effort_limit" value="0.5"/>
   <xacro:property name="shoulder_lower" value="-${default_joint_position_limit}"/>
   <xacro:property name="shoulder_upper" value="${default_joint_position_limit}"/>

File: ros_ws/src/pingu_description/urdf/arms/levion_arm.ros2_control.xacro (robot description, xacro)
@@ -1,7 +1,8 @@
 <?xml version="1.0"?>
 <robot xmlns:xacro="http://www.ros.org/wiki/xacro">
-<xacro:macro name="levion_system" params="name prefix left_arm:=true right_arm:=false hw_plugin:='real'"> <!-- real/mujoco-->
+<xacro:macro name="levion_system" params="name prefix left_arm:=true right_arm:=false hw_plugin:='real'"> <!-- real/mit/mujoco/gazebo -->
 <!-- include macros -->
 <xacro:include filename="arms/ak80_8.macros.xacro"/>
+<xacro:include filename="$(find cubemars_mit_hardware)/ros2_control/ak80_8_mit.macros.xacro"/>
 <xacro:include filename="arms/levion.property.xacro"/>
 <ros2_control name="${name}" type="system">
@@ -9,4 +10,10 @@
     <hardware>
       <plugin>cubemars_hardware/CubeMarsSystemHardware</plugin>
+      <param name="can_interface">can0</param>
+    </hardware>
+  </xacro:if>
+  <xacro:if value="${hw_plugin == 'mit'}">
+    <hardware>
+      <plugin>cubemars_mit_hardware/MITHardwareInterface</plugin>
       <param name="can_interface">can0</param>
     </hardware>
@@ -22,9 +29,9 @@
     </hardware>
   </xacro:if>
-  <!-- Left arm -->
-  <xacro:if value="${left_arm}">
+  <!-- Left arm (servo mode) -->
+  <xacro:if value="${left_arm and hw_plugin != 'mit'}">
     <xacro:ak80_8_ros2_control
       joint_name="${prefix}left_shoulder_joint"
-      can_id="104"
+      can_id="204"
       pos_min="${left_shoulder_lower}"
       pos_max="${left_shoulder_upper}"
@@ -41,9 +48,26 @@
       enc_off="${left_elbow_enc_offset}"/>
   </xacro:if>
-  <!-- Right arm -->
-  <xacro:if value="${right_arm}">
+  <!-- Left arm (MIT mode) -->
+  <xacro:if value="${left_arm and hw_plugin == 'mit'}">
+    <xacro:ak80_8_mit_ros2_control
+      joint_name="${prefix}left_shoulder_joint"
+      can_id="204"
+      pos_min="${left_shoulder_lower}"
+      pos_max="${left_shoulder_upper}"
+      vel_limit="${left_shoulder_velocity_limit}"
+      effort_limit="${left_shoulder_effort_limit}"/>
+    <xacro:ak80_8_mit_ros2_control
+      joint_name="${prefix}left_elbow_joint"
+      can_id="105"
+      pos_min="${left_elbow_lower}"
+      pos_max="${left_elbow_upper}"
+      vel_limit="${left_elbow_velocity_limit}"
+      effort_limit="${left_elbow_effort_limit}"/>
+  </xacro:if>
+  <!-- Right arm (servo mode) -->
+  <xacro:if value="${right_arm and hw_plugin != 'mit'}">
     <xacro:ak80_8_ros2_control
       joint_name="${prefix}right_shoulder_joint"
-      can_id="204"
+      can_id="104"
       pos_min="${right_shoulder_lower}"
       pos_max="${right_shoulder_upper}"
@@ -60,4 +84,21 @@
       enc_off="${right_elbow_enc_offset}"/>
   </xacro:if>
+  <!-- Right arm (MIT mode) -->
+  <xacro:if value="${right_arm and hw_plugin == 'mit'}">
+    <xacro:ak80_8_mit_ros2_control
+      joint_name="${prefix}right_shoulder_joint"
+      can_id="104"
+      pos_min="${right_shoulder_lower}"
+      pos_max="${right_shoulder_upper}"
+      vel_limit="${right_shoulder_velocity_limit}"
+      effort_limit="${right_shoulder_effort_limit}"/>
+    <xacro:ak80_8_mit_ros2_control
+      joint_name="${prefix}right_elbow_joint"
+      can_id="205"
+      pos_min="${right_elbow_lower}"
+      pos_max="${right_elbow_upper}"
+      vel_limit="${right_elbow_velocity_limit}"
+      effort_limit="${right_elbow_effort_limit}"/>
+  </xacro:if>
 </ros2_control>
 </xacro:macro>

File: ros_ws/src/pingu_description/urdf/pingu.urdf.xacro (robot description, xacro)
@@ -8,4 +8,8 @@
   <xacro:arg name="left_arm" default="true" />        <!-- Enable left arm -->
   <xacro:arg name="right_arm" default="true" />       <!-- Enable right arm -->
+  <xacro:arg name="left_shoulder" default="true" />   <!-- Enable left shoulder motor -->
+  <xacro:arg name="left_elbow" default="true" />      <!-- Enable left elbow motor -->
+  <xacro:arg name="right_shoulder" default="true" />  <!-- Enable right shoulder motor -->
+  <xacro:arg name="right_elbow" default="true" />     <!-- Enable right elbow motor -->
   <!-- Check if it has arms-->
   <xacro:property name="has_arm" value="false"/>
@@ -93,4 +97,8 @@
         left_arm="$(arg left_arm)"
         right_arm="$(arg right_arm)"
+        left_shoulder="$(arg left_shoulder)"
+        left_elbow="$(arg left_elbow)"
+        right_shoulder="$(arg right_shoulder)"
+        right_elbow="$(arg right_elbow)"
         hw_plugin="$(arg hw_plugin)"/>
     </xacro:if>

File: ros_ws/src/rw_ros2_control/description/ros2_control/rw.ros2_control.xacro (robot description, xacro)
@@ -4,5 +4,6 @@
     <ros2_control name="${name}" type="system">
       <!-- Chose hardware interfaces -->
-      <xacro:if value="${hw_plugin == 'real'}">
+      <!-- rsl_servo only changes the ARM driver; the reaction wheel stays on ODrive -->
+      <xacro:if value="${hw_plugin == 'real' or hw_plugin == 'rsl_servo'}">
         <hardware>
           <plugin>odrive_ros2_control_plugin/ODriveHardwareInterface</plugin>
